File: TPA3116/KAmp_TPA3116D2.kicad_pcb (KiCad board)
At the start: 2 copper layers, 100 x 60 mm, 280 parts, among them J1 CTRL, J2 R_IN, J3 L_IN, J4 Sync, J5 Sync, J6 R_OUT, J7 Barrel_Jack_Switch, J8 L_OUT, U1 TPA3116D2

Commit message: 将端子向板边延伸2mm
Parts:
- J1: footprint Connector_PinHeader_2.54mm:PinHeader_1x04_P2.54mm_Vertical -> Connector_Molex:Molex_KK-254_AE-6410-04A_1x04_P2.54mm_Vertical
- J2, J3, J4, J5: footprint Connector_PinHeader_2.54mm:PinHeader_1x02_P2.54mm_Vertical -> Connector_Molex:Molex_KK-254_AE-6410-02A_1x02_P2.54mm_Vertical
- moved J4 3.71 mm to (68.5, 107.9), turned to 90 degrees
- moved J5 3.54 mm to (68.5, 101.8), turned to 90 degrees
- moved J7 2.78 mm to (138.6, 66.1)
- moved J6 2.20 mm to (142.0, 82.4)
- moved J8 2.20 mm to (142.0, 96.7)
- moved J1 0.65 mm to (56.9, 72.5), turned to 90 degrees
- moved J3 0.55 mm to (57.0, 95.0), turned to 90 degrees
- moved J2 0.36 mm to (57.1, 84.9), turned to 90 degrees
Routing:
- net +24V: track 135.6 -> 138.8 mm
